File: xilinxtest/xilinxtest.sch (KiCad schematic (older format))
At the start: 26 parts, among them U1 XC7A35T-CPG236

Commit message: Added some power components
Parts:
- added C? (x7): 47nF, symbol Device:C
- added C? (x3): 47uF, symbol Device:C
- added C? (x6): 470nF, symbol Device:C
- added C? (x5): 4.7uF, symbol Device:C
- added C? (x3): 100uF, symbol Device:C
Connections:
- net labels added: VCC1V0, VCC1V8
- wire segments 143 -> 300

Commit message: associated all footprints
Parts:
- removed C?: 100uF, symbol Device:C
- added C? (x2): 47nF, Capacitor_SMD:C_0805_2012Metric, symbol Device:C
- added C? (x2): 470nF, Capacitor_SMD:C_0805_2012Metric, symbol Device:C
- added C?: 4.7uF, Capacitor_SMD:C_0805_2012Metric, symbol Device:C
- added C?: 100uF, Capacitor_SMD:C_1210_3225Metric, symbol Device:C
- added C?: 4.7nF, Capacitor_SMD:C_0805_2012Metric, symbol Device:C
- C? (x25): footprint (none) -> Capacitor_SMD:C_0805_2012Metric
- C? (x2): footprint (none) -> Capacitor_SMD:C_1210_3225Metric
- FlashMemory: footprint (none) -> Package_DIP:DIP-8_W7.62mm
- J?: footprint (none) -> Connector_PinHeader_2.00mm:PinHeader_2x07_P2.00mm_Vertical
- R? (x18): footprint (none) -> Resistor_SMD:R_0805_2012Metric
Connections:
- wire segments 300 -> 343

Commit message: Started on PCB Layout
Parts:
- added C10: 10uF, Capacitor_SMD:C_0805_2012Metric, symbol Device:C_Small
- added C12, C23, C5, C9: 0.1uF, Capacitor_SMD:C_0805_2012Metric, symbol Device:C_Small
- added C25, C31, C45, C46, C49, C50: 2.2uF, Capacitor_SMD:C_0805_2012Metric, symbol Device:C
- added C37, C38, C39, C42, C43, C55, C56, C61, C62, C64: 100nF, Capacitor_SMD:C_0805_2012Metric, symbol Device:C_Small
- added C47, C48, C53, C54: 100uF, Capacitor_SMD:C_1210_3225Metric, symbol Device:C_Small
- added C51, C52, C58, C59: 47uF, Capacitor_SMD:C_0805_2012Metric, symbol Device:C_Small
- added C6: 1uF, Capacitor_SMD:C_0805_2012Metric, symbol Device:C_Small
- added D2: LG R971, LED_SMD:LED_0805_2012Metric, symbol LED:SFH4346
- added J2: -INPUT, Connector_PinHeader_2.54mm:PinHeader_1x01_P2.54mm_Vertical, symbol Connector:Conn_01x01_Female
- added J3: GNDJUMP, Connector_PinHeader_2.54mm:PinHeader_1x02_P2.54mm_Vertical, symbol Connector:Conn_01x02_Female
- added J4: +INPUT, Connector_PinHeader_2.54mm:PinHeader_1x01_P2.54mm_Vertical, symbol Connector:Conn_01x01_Female
- added J5: OutputGND, Connector_PinHeader_2.54mm:PinHeader_1x01_P2.54mm_Vertical, symbol Connector:Conn_01x01_Female
- added J6: 5V_SUPPLY, Connector_PinSocket_2.54mm:PinSocket_1x01_P2.54mm_Vertical, symbol Connector:Conn_01x01_Female
- added J7: GND_SUPPLY, Connector_PinSocket_2.54mm:PinSocket_1x01_P2.54mm_Vertical, symbol Connector:Conn_01x01_Female
- added L1, L2, L3, L4: 1.5u, Inductor_SMD:L_7.3x7.3_H4.5, symbol Device:L
- added Q1: FDV301N, Package_TO_SOT_SMD:SOT-23, symbol Device:Q_NMOS_GSD
- added R10, R11, R2, R21, R22, R23, R24, R25, R26, R27, R28, R29, R3, R30, R31, R32, R33, R34, R35, R36, R37, R38, R39, R4, R49, R5, R50, R51, R52, R53, R54, R55, R56, R57, R58, R59, R6, R60, R61, R62, R63, R64: 100, Resistor_SMD:R_0805_2012Metric, symbol Device:R
- added R45, R48: 100k, Resistor_SMD:R_0805_2012Metric, symbol Device:R_US
- added R46, R47: 200k, Resistor_SMD:R_0805_2012Metric, symbol Device:R_US
- added R65, R68: 13.3k, Resistor_SMD:R_0805_2012Metric, symbol Device:R_US
- added R66, R67, R70, R71: 60.4k, Resistor_SMD:R_0805_2012Metric, symbol Device:R_US
- added R69: 90.9k, Resistor_SMD:R_0805_2012Metric, symbol Device:R_US
- added R72: 30.1k, Resistor_SMD:R_0805_2012Metric, symbol Device:R_US
- added R73, R75, R77: 10k, Resistor_SMD:R_0805_2012Metric, symbol Device:R_US
- added R74: 4.7k, Resistor_SMD:R_0805_2012Metric, symbol Device:R_US
- added R76: 680, Resistor_SMD:R_0805_2012Metric, symbol Device:R_US
- added SW1: SW_SPDT, SPDT:SPDTSwitch, symbol Switch:SW_SPDT
- added U2: ADS8412, Package_QFP:LQFP-48_7x7mm_P0.5mm, symbol CaseysParts:ADS8412
- added U3: LTC1657, Package_SO:SSOP-28_3.9x9.9mm_P0.635mm, symbol CaseysParts:LTC1657
- added U4, U5: LTC3633-TSSOP, Package_SO:TSSOP-28-1EP_4.4x9.7mm_P0.65mm, symbol FPGA_Power_Project:LTC3633-TSSOP
- D1: renamed from D?; footprint (none) -> Diode_SMD:D_0805_2012Metric
- gave numbers to parts that had none: 53
- renumbered FlashMemory to FlashMemory1
Connections:
- net labels added: 5V, ADCBUSY, ADCCS, ADCRESET, AGND, ASYNCHDAC, BDGND, CONVSTART, D0, D1, D10, D11, D12, D13, D14, D15, D2, D3, D4, D5, D6, D7, D8, D9, DACCLR, DACWRITE, DAC_out, DB0, DB1, DB10, DB11, DB12, DB13, DB14, DB15, DB2, DB3, DB4, DB5, DB6, DB7, DB8, DB9, EN, LEDPWRUP, OUTENABLE, VCC3V3ADCFLASH, VCC3V3FPGA
- wire segments 343 -> 686
